File: hardware/TUSS4470_shield/TUSS4470_shield/TUSS4470_shield.kicad_pcb (KiCad board)
At the start: 2 copper layers, 69 x 53.8 mm, 35 parts, among them J1 VIN, J2 TRANSDUCER, J3 Conn_01x10_Socket, J4 VCC SELECT, J5 Conn_01x08_Socket, J6 Conn_01x06_Socket, J7 Conn_01x08_Socket, SW1 RST, U1 TUSS4470TRTJR

Commit message: fixed fooprint c3 and minor design changes
Parts:
- C3: footprint Capacitor_SMD:C_0201_0603Metric -> Capacitor_SMD:C_0603_1608Metric
- moved C3 0.89 mm to (121.4, 49.6)
- moved C1 0.42 mm to (121.4, 45.5)
Routing:
- net GND: track 25.9 -> 27.7 mm
Other:
- board text added: "PIN | TUSS4470 5 | OUT_4 6 | OUT_3 8 | IO_1 9 | IO_2 10 | CS 11 | DI 12 | DO 13 | CLK A0 | VOUT"
- board text added: "cFLT"
- board text added: "cINN"
- board text removed: "G"
- board text removed: "PIN | FUNCTION 5 | OUT_4 6 | OUT_3 8 | IO_1 9 | IO_2 10 | CS 11 | DI 12 | DO 13 | CLK A0 | VOUT"
