File: TUSS4470_shield_002/TUSS4470_shield_hardware/TUSS4470_shield/TUSS4470_shield.kicad_pcb (KiCad board)
At the start: 2 copper layers, 69 x 53.8 mm, 36 parts, among them J1 VIN, J2 TRANSDUCER, J3 Conn_01x10_Socket, J4 VCC SELECT, J5 Conn_01x08_Socket, J6 Conn_01x06_Socket, J7 Conn_01x08_Socket, J8 Conn_01x02_Pin, SW1 RST, U1 TUSS4470TRTJR

Commit message: added latest version 2 files for production run 2
Parts:
- C10: value CXXnF -> 8.2nF
- C9: value CXXnF -> 1nF
Other:
- board text added: "ver: 002 2025-05-02"
- board text removed: "ver: 002 2025-03-27"
