File: TUSS4470_shield_002/TUSS4470_shield_hardware/TUSS4470_shield/TUSS4470_shield.kicad_sch (KiCad schematic)
At the start: 36 parts, among them J1 VIN, J2 TRANSDUCER, J3 Conn_01x10_Socket, J4 VCC SELECT, J5 Conn_01x08_Socket, J6 Conn_01x06_Socket, J7 Conn_01x08_Socket, J8 Conn_01x02_Pin, SW1 RST, U1 TUSS4470TRTJR

Commit message: added latest version 2 files for production run 2
Parts:
- C10: value CXXnF -> 8.2nF; LCSC (none) -> C1322360; now fitted; now in the parts list
- C9: value CXXnF -> 1nF; LCSC (none) -> C1588; now fitted; now in the parts list
- J1: LCSC (none) -> C431092; now fitted; now in the parts list
- J4: LCSC (none) -> C49257; now fitted; now in the parts list
- JP1, JP2, JP3, JP4, JP5, JP6: LCSC (none) -> C2905434; now fitted; now in the parts list
Other:
- note added: "1nF is used for combination with 200kHz (3.2nF) to achieve 150kHz"
- note added: "8.2nF is used for combination with 200kHz (21.2nF) to achieve 150kHz"
Changed lines of the file:
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@@
 (kicad_sch
-	(version 20231120)
+	(version 20250114)
 	(generator "eeschema")
-	(generator_version "8.0")
+	(generator_version "9.0")
 	(paper "A4")
+	(text "8.2nF is used for \ncombination with \n200kHz (21.2nF) \nto achieve 150kHz"
+		(exclude_from_sim no)
+		(at 29.718 85.344 0)
+		(effects
+			(font
+				(size 1.27 1.27)
+			)
+		)
+	)
+	(text "1nF is used for \ncombination with \n200kHz (3.2nF) \nto achieve 150kHz"
+		(exclude_from_sim no)
+		(at 54.356 109.474 0)
+		(effects
+			(font
+				(size 1.27 1.27)
+			)
+		)
+	)
+	(text_box "cFLT"
+		(exclude_from_sim no)
+		(at 53.34 99.06 0)
+		(size 12.7 2.54)
+		(margins 0.9525 0.9525 0.9525 0.9525)
+		(stroke
+			(width 0)
+			(type default)
+		)
+		(fill
+			(type none)
+		)
+		(effects
+			(font
+				(size 1.27 1.27)
+			)
+			(justify left top)
+		)
+	)
+	(text_box "For frequencies other than 40kHz or 200kHz see datasheet page 31:\nhttps://www.ti.com/lit/ds/symlink/tuss4470.pdf"
+		(exclude_from_sim no)
+		(at 40.64 127 0)
+		(size 53.34 10.16)
+		(margins 0.9525 0.9525 0.9525 0.9525)
+		(stroke
+			(width 0)
+			(type default)
+		)
+		(fill
+			(type none)
+		)
+		(effects
+			(font
+				(size 1.27 1.27)
+			)
+			(justify left top)
+		)
+	)
+	(text_box "cINN"
+		(exclude_from_sim no)
+		(at 22.86 73.66 0)
+		(size 15.24 2.54)
+		(margins 0.9525 0.9525 0.9525 0.9525)
+		(stroke
+			(width 0)
+			(type default)
+		)
+		(fill
+			(type none)
+		)
+		(effects
+			(font
+				(size 1.27 1.27)
+			)
+			(justify left top)
+		)
+	)
 	(junction
 		(at 237.49 27.94)
@@
 		)
 	)
-	(text_box "cFLT"
-		(exclude_from_sim no)
-		(at 53.34 99.06 0)
-		(size 12.7 2.54)
-		(stroke
-			(width 0)
-			(type default)
-		)
-		(fill
-			(type none)
-		)
-		(effects
-			(font
-				(size 1.27 1.27)
-			)
-			(justify left top)
-		)
-	)
-	(text_box "For frequencies other than 40kHz or 200kHz see datasheet page 31:\nhttps://www.ti.com/lit/ds/symlink/tuss4470.pdf"
-		(exclude_from_sim no)
-		(at 40.64 127 0)
-		(size 53.34 10.16)
-		(stroke
-			(width 0)
-			(type default)
-		)
-		(fill
-			(type none)
-		)
-		(effects
-			(font
-				(size 1.27 1.27)
-			)
-			(justify left top)
-		)
-	)
-	(text_box "cINN"
-		(exclude_from_sim no)
-		(at 22.86 73.66 0)
-		(size 15.24 2.54)
-		(stroke
-			(width 0)
-			(type default)
-		)
-		(fill
-			(type none)
-		)
-		(effects
-			(font
-				(size 1.27 1.27)
-			)
-			(justify left top)
-		)
-	)
 	(global_label "NCS"
 		(shape input)
@@
 		(unit 1)
 		(exclude_from_sim no)
-		(in_bom no)
+		(in_bom yes)
 		(on_board yes)
-		(dnp yes)
+		(dnp no)
 		(fields_autoplaced yes)
 		(property "Reference" "C9"
@@
 			)
 		)
-		(property "Value" "CXXnF"
+		(property "Value" "1nF"
 			(at 71.12 114.2999 0)
 			(effects
@@
 			)
 		)
+		(property "LCSC" "C1588"
+			(at 67.31 113.03 0)
+			(effects
+				(font
+					(size 1.27 1.27)
+				)
+				(hide yes)
+			)
+		)
 		(pin "1"
 		)
@@
 		(at 55.88 78.74 90)
 		(unit 1)
-		(exclude_from_sim yes)
-		(in_bom no)
+		(exclude_from_sim no)
+		(in_bom yes)
 		(on_board yes)
-		(dnp yes)
+		(dnp no)
 		(fields_autoplaced yes)
 		(property "Reference" "JP2"
@@
 			)
 		)
+		(property "LCSC" "C2905434"
+			(at 55.88 78.74 90)
+			(effects
+				(font
+					(size 1.27 1.27)
+				)
+				(hide yes)
+			)
+		)
 		(pin "2"
 		)
@@
 		(unit 1)
 		(exclude_from_sim no)
-		(in_bom no)
+		(in_bom yes)
 		(on_board yes)
-		(dnp yes)
+		(dnp no)
 		(fields_autoplaced yes)
 		(property "Reference" "C10"
@@
 			)
 		)
-		(property "Value" "CXXnF"
+		(property "Value" "8.2nF"
 			(at 44.45 87.6299 0)
 			(effects
@@
 			)
 		)
+		(property "LCSC" "C1322360"
+			(at 40.64 86.36 0)
+			(effects
+				(font
+					(size 1.27 1.27)
+				)
+				(hide yes)
+			)
+		)
 		(pin "1"
 		)
@@
 		(unit 1)
 		(exclude_from_sim no)
-		(in_bom no)
+		(in_bom yes)
 		(on_board yes)
-		(dnp yes)
+		(dnp no)
 		(fields_autoplaced yes)
 		(property "Reference" "J1"
@@
 			)
 		)
+		(property "LCSC" "C431092"
+			(at 252.73 21.59 90)
+			(effects
+				(font
+					(size 1.27 1.27)
+				)
+				(hide yes)
+			)
+		)
 		(pin "2"
 		)
@@
 		(at 71.12 78.74 90)
 		(unit 1)
-		(exclude_from_sim yes)
-		(in_bom no)
+		(exclude_from_sim no)
+		(in_bom yes)
 		(on_board yes)
-		(dnp yes)
+		(dnp no)
 		(fields_autoplaced yes)
 		(property "Reference" "JP4"
@@
 			)
 		)
+		(property "LCSC" "C2905434"
+			(at 71.12 78.74 90)
+			(effects
+				(font
+					(size 1.27 1.27)
+				)
+				(hide yes)
+			)
+		)
 		(pin "2"
 		)
@@
 		(at 67.31 105.41 90)
 		(unit 1)
-		(exclude_from_sim yes)
-		(in_bom no)
+		(exclude_from_sim no)
+		(in_bom yes)
 		(on_board yes)
-		(dnp yes)
+		(dnp no)
 		(property "Reference" "JP5"
 			(at 69.85 104.1399 90)
@@
 			)
 		)
+		(property "LCSC" "C2905434"
+			(at 67.31 105.41 90)
+			(effects
+				(font
+					(size 1.27 1.27)
+				)
+				(hide yes)
+			)
+		)
 		(pin "2"
 		)
@@
 		(at 40.64 78.74 90)
 		(unit 1)
-		(exclude_from_sim yes)
-		(in_bom no)
+		(exclude_from_sim no)
+		(in_bom yes)
 		(on_board yes)
-		(dnp yes)
+		(dnp no)
 		(property "Reference" "JP6"
 			(at 43.18 77.4699 90)
@@
 			)
 		)
+		(property "LCSC" "C2905434"
+			(at 40.64 78.74 90)
+			(effects
+				(font
+					(size 1.27 1.27)
+				)
+				(hide yes)
+			)
+		)
 		(pin "2"
 		)
@@
 		(at 95.25 105.41 90)
 		(unit 1)
-		(exclude_from_sim yes)
-		(in_bom no)
+		(exclude_from_sim no)
+		(in_bom yes)
 		(on_board yes)
-		(dnp yes)
+		(dnp no)
 		(fields_autoplaced yes)
 		(property "Reference" "JP3"
@@
 			)
 		)
+		(property "LCSC" "C2905434"
+			(at 95.25 105.41 90)
+			(effects
+				(font
+					(size 1.27 1.27)
+				)
+				(hide yes)
+			)
+		)
 		(pin "2"
 		)
@@
 		(unit 1)
 		(exclude_from_sim no)
-		(in_bom no)
+		(in_bom yes)
 		(on_board yes)
-		(dnp yes)
+		(dnp no)
 		(fields_autoplaced yes)
 		(property "Reference" "J4"
@@
 			)
 		)
+		(property "LCSC" "C49257"
+			(at 240.03 21.59 90)
+			(effects
+				(font
+					(size 1.27 1.27)
+				)
+				(hide yes)
+			)
+		)
 		(pin "3"
 		)
@@
 		(at 81.28 105.41 90)
 		(unit 1)
-		(exclude_from_sim yes)
-		(in_bom no)
+		(exclude_from_sim no)
+		(in_bom yes)
 		(on_board yes)
-		(dnp yes)
+		(dnp no)
 		(fields_autoplaced yes)
 		(property "Reference" "JP1"
@@
 			)
 		)
+		(property "LCSC" "C2905434"
+			(at 81.28 105.41 90)
+			(effects
+				(font
+					(size 1.27 1.27)
+				)
+				(hide yes)
+			)
+		)
 		(pin "2"
 		)
@@
 		)
 	)
+	(embedded_fonts no)
 )
